Commit message: add support for payload and spring payload to GVR

File: dynamics/resources/gvr_bot/gvrbot_updated_tmp.urdf (robot description, URDF)
Before this commit: robot gvrbot_updated, 25 links, 24 joints
Links:
- added link payload_block_0, mass 2.0; collision box size=0.15 0.15 0.05; visual box size=0.15 0.15 0.05
- added link payload_block_1, mass 2.0; collision box size=0.15 0.15 0.05; visual box size=0.15 0.15 0.05
- added link payload_block_2, mass 2.0; collision box size=0.15 0.15 0.05; visual box size=0.15 0.15 0.05
- added link payload_block_3, mass 2.0; collision box size=0.15 0.15 0.05; visual box size=0.15 0.15 0.05
- added link payload_block_4, mass 2.0; collision box size=0.15 0.15 0.05; visual box size=0.15 0.15 0.05
- added link payload_block_5, mass 2.0; collision box size=0.15 0.15 0.05; visual box size=0.15 0.15 0.05
- added link payload_block_6, mass 2.0; collision box size=0.15 0.15 0.05; visual box size=0.15 0.15 0.05
- added link payload_block_7, mass 2.0; collision box size=0.15 0.15 0.05; visual box size=0.15 0.15 0.05
- added link payload_block_8, mass 2.0; collision box size=0.15 0.15 0.05; visual box size=0.15 0.15 0.05
- added link payload_block_9, mass 2.0; collision box size=0.15 0.15 0.05; visual box size=0.15 0.15 0.05
Joints:
- added joint body_payload: type fixed, parent base_link, child payload_block_0
- added joint payload0_payload1: type revolute, parent payload_block_0, child payload_block_1, origin xyz=0.0 0.0 0.05 rpy=0 0 0.0, axis 0 1 0, limit lower=-0.5 upper=0.5 effort=10.0 velocity=10.0
- added joint payload1_payload2: type revolute, parent payload_block_1, child payload_block_2, origin xyz=0.0 0.0 0.05 rpy=0 0 0.0, axis 1 0 0, limit lower=-0.5 upper=0.5 effort=10.0 velocity=10.0
- added joint payload2_payload3: type revolute, parent payload_block_2, child payload_block_3, origin xyz=0.0 0.0 0.05 rpy=0 0 0.0, axis 0 1 0, limit lower=-0.5 upper=0.5 effort=10.0 velocity=10.0
- added joint payload3_payload4: type revolute, parent payload_block_3, child payload_block_4, origin xyz=0.0 0.0 0.05 rpy=0 0 0.0, axis 1 0 0, limit lower=-0.5 upper=0.5 effort=10.0 velocity=10.0
- added joint payload4_payload5: type revolute, parent payload_block_4, child payload_block_5, origin xyz=0.0 0.0 0.05 rpy=0 0 0.0, axis 0 1 0, limit lower=-0.5 upper=0.5 effort=10.0 velocity=10.0
- added joint payload5_payload6: type revolute, parent payload_block_5, child payload_block_6, origin xyz=0.0 0.0 0.05 rpy=0 0 0.0, axis 1 0 0, limit lower=-0.5 upper=0.5 effort=10.0 velocity=10.0
- added joint payload6_payload7: type revolute, parent payload_block_6, child payload_block_7, origin xyz=0.0 0.0 0.05 rpy=0 0 0.0, axis 0 1 0, limit lower=-0.5 upper=0.5 effort=10.0 velocity=10.0
- added joint payload7_payload8: type revolute, parent payload_block_7, child payload_block_8, origin xyz=0.0 0.0 0.05 rpy=0 0 0.0, axis 1 0 0, limit lower=-0.5 upper=0.5 effort=10.0 velocity=10.0
- added joint payload8_payload9: type revolute, parent payload_block_8, child payload_block_9, origin xyz=0.0 0.0 0.05 rpy=0 0 0.0, axis 0 1 0, limit lower=-0.5 upper=0.5 effort=10.0 velocity=10.0

Commit message: calibrate spring payload to result in more failures

File: dynamics/resources/gvr_bot/gvrbot_updated_tmp.urdf (robot description, URDF)
Before this commit: robot gvrbot_updated, 35 links, 34 joints
Links:
- removed link payload_block_6
- removed link payload_block_7
- removed link payload_block_8
- removed link payload_block_9
- link payload_block_0: mass 2.0 -> 8.333333333333334; geometry collision box size=0.15 0.15 0.2; visual box size=0.15 0.15 0.2
- link payload_block_1: mass 2.0 -> 8.333333333333334; geometry collision box size=0.15 0.15 0.2; visual box size=0.15 0.15 0.2
- link payload_block_2: mass 2.0 -> 8.333333333333334; geometry collision box size=0.15 0.15 0.2; visual box size=0.15 0.15 0.2
- link payload_block_3: mass 2.0 -> 8.333333333333334; geometry collision box size=0.15 0.15 0.2; visual box size=0.15 0.15 0.2
- link payload_block_4: mass 2.0 -> 8.333333333333334; geometry collision box size=0.15 0.15 0.2; visual box size=0.15 0.15 0.2
- link payload_block_5: mass 2.0 -> 8.333333333333334; geometry collision box size=0.15 0.15 0.2; visual box size=0.15 0.15 0.2
Joints:
- removed joint payload5_payload6
- removed joint payload6_payload7
- removed joint payload7_payload8
- removed joint payload8_payload9
- joint payload0_payload1: limit lower=-0.5 upper=0.5 effort=10.0 velocity=10.0 -> lower=-0.5 upper=0.5 effort=10.0 velocity=20.0; origin xyz=0.0 0.0 0.05 rpy=0 0 0.0 -> xyz=0.0 0.0 0.2 rpy=0 0 0.0
- joint payload1_payload2: limit lower=-0.5 upper=0.5 effort=10.0 velocity=10.0 -> lower=-0.5 upper=0.5 effort=10.0 velocity=20.0; origin xyz=0.0 0.0 0.05 rpy=0 0 0.0 -> xyz=0.0 0.0 0.2 rpy=0 0 0.0
- joint payload2_payload3: limit lower=-0.5 upper=0.5 effort=10.0 velocity=10.0 -> lower=-0.5 upper=0.5 effort=10.0 velocity=20.0; origin xyz=0.0 0.0 0.05 rpy=0 0 0.0 -> xyz=0.0 0.0 0.2 rpy=0 0 0.0
- joint payload3_payload4: limit lower=-0.5 upper=0.5 effort=10.0 velocity=10.0 -> lower=-0.5 upper=0.5 effort=10.0 velocity=20.0; origin xyz=0.0 0.0 0.05 rpy=0 0 0.0 -> xyz=0.0 0.0 0.2 rpy=0 0 0.0
- joint payload4_payload5: limit lower=-0.5 upper=0.5 effort=10.0 velocity=10.0 -> lower=-0.5 upper=0.5 effort=10.0 velocity=20.0; origin xyz=0.0 0.0 0.05 rpy=0 0 0.0 -> xyz=0.0 0.0 0.2 rpy=0 0 0.0
