Commit message: add flag to turn on/off flippers

File: dynamics/resources/gvr_bot/gvrbot_updated.urdf (robot description, URDF)
Before this commit: robot gvrbot_updated, 25 links, 24 joints
Links:
- removed link LF_flipper_main
- removed link RF_flipper_main
Joints:
- removed joint base_to_LF_flipper
- removed joint base_to_RF_flipper

File: dynamics/resources/gvr_bot/gvrbot_updated_tmp.urdf (robot description, URDF)
Before this commit: robot gvrbot_updated, 31 links, 30 joints
Links:
- removed link LF_flipper_main
- removed link RF_flipper_main
- removed link payload_block_0
- removed link payload_block_1
- removed link payload_block_2
- removed link payload_block_3
- removed link payload_block_4
- removed link payload_block_5
- added link sail_base, mass 1.0; collision box size=0.03 0.05 0.90; visual box size=0.03 0.05 0.90
- added link sail_panel, mass 1.0; collision box size=0.9 0.02 0.8; visual box size=0.9 0.02 0.8
Joints:
- removed joint base_to_LF_flipper
- removed joint base_to_RF_flipper
- removed joint payload0_payload1
- removed joint payload1_payload2
- removed joint payload2_payload3
- removed joint payload3_payload4
- removed joint payload4_payload5
- added joint sail_connector: type fixed, parent sail_base, child sail_panel
- joint body_payload: child payload_block_0 -> sail_base

Commit message: fix simulator with user's action instead of explicit control, fix to use latest URDF from Peraton

File: dynamics/resources/gvr_bot/gvrbot_updated.urdf (robot description, URDF)
Before this commit: robot gvrbot_updated, 23 links, 22 joints
Links:
- added link 1010_base, mass 0.325; visual box size=0.0254 0.0254 0.430
- added link 1020_base, mass 0.589; visual box size=0.0508 0.0254 0.430
- added link LF_flipper_main, mass 1.026; collision mesh filename=flipper.stl scale=0.001 0.001 0.001; visual mesh filename=flipper.stl scale=0.001 0.001 0.001
- added link RF_flipper_main, mass 1.026; collision mesh filename=flipper.stl scale=0.001 0.001 0.001; visual mesh filename=flipper.stl scale=0.001 0.001 0.001
- added link back_staff, mass 0.577; visual box size=0.0254 0.0254 0.762
- added link bottom_bar, mass 0.692; visual box size=0.0254 0.0254 0.914
- added link front_staff, mass 1.3937; visual box size=0.0508 0.0254 1.016
- added link little_piece, mass 0.0769; visual box size=0.0254 0.0254 0.1016
- added link top_bar, mass 0.692; visual box size=0.0254 0.0254 0.914
- link L1: mass 0.06227 -> 0.12455
- link L10: mass 0.06227 -> 0.12455
- link L11: mass 0.06227 -> 0.12455
- link L2: mass 0.06227 -> 0.12455
- link L3: mass 0.06227 -> 0.12455
- link L4: mass 0.06227 -> 0.12455
- link L5: mass 0.06227 -> 0.12455
- link L6: mass 0.06227 -> 0.12455
- link L7: mass 0.06227 -> 0.12455
- link L8: mass 0.06227 -> 0.12455
- link L9: mass 0.06227 -> 0.12455
- link R1: mass 0.06227 -> 0.12455
- link R10: mass 0.06227 -> 0.12455
- link R11: mass 0.06227 -> 0.12455
- link R2: mass 0.06227 -> 0.12455
- link R3: mass 0.06227 -> 0.12455
- link R4: mass 0.06227 -> 0.12455
- link R5: mass 0.06227 -> 0.12455
- link R6: mass 0.06227 -> 0.12455
- link R7: mass 0.06227 -> 0.12455
- link R8: mass 0.06227 -> 0.12455
- link R9: mass 0.06227 -> 0.12455
- link base_link: mass 16.9 -> 16.4; geometry collision box size=0.588 0.254 0.06; visual mesh filename=Base_Centered_Stripped.obj scale=1.0 1.0 1.0
Joints:
- added joint 1010_base_to_little_piece: type fixed, parent 1010_base, child little_piece, origin xyz=0 0 0.0635
- added joint 1020_base_to_front_staff: type fixed, parent 1020_base, child front_staff, origin xyz=0 0 0.5207
- added joint base_to_1010_base: type fixed, parent base_link, child 1010_base, origin xyz=-0.2973 0 0.12
- added joint base_to_1020_base: type fixed, parent base_link, child 1020_base, origin xyz=0.248 0 0.12
- added joint base_to_RF_flipper: type continuous, parent base_link, child RF_flipper_main, origin xyz=0.2605 0.2418 0.0125, axis 0 1 0, limit effort=1.0 velocity=0.5
- added joint base_to_flippers: type continuous, parent base_link, child LF_flipper_main, origin xyz=0.2605 -0.2418 0.0125, axis 0 1 0, limit effort=1.0 velocity=1.2
- added joint bottom_bar: type fixed, parent bottom_bar, child top_bar, origin xyz=0 0 0.7854
- added joint bottom_bar_to_back_staff: type fixed, parent bottom_bar, child back_staff, origin xyz=-0.3693 0 0.3937
- added joint front_staff_to_bottom_bar: type fixed, parent front_staff, child bottom_bar, origin xyz=-0.4761 0 -0.4064

File: dynamics/resources/gvr_bot/test_track/Block/Terrain_Test_Block.urdf (robot description, URDF)
Before this commit: robot Terrain_Test_Block.urdf, 1 links, 0 joints
Links:
- removed link Terrain_Block
- added link block, mass 1000.0; collision mesh filename=./Terrain_Test_Block_meters.obj scale=1.0 1.0 1.0; visual mesh filename=./Terrain_Test_Block_meters.obj scale=1.0 1.0 1.0
- added link world
Joints:
- added joint ramp_to_plane: type fixed, parent world, child block, origin xyz=0 0 0 rpy=1.57079 0 0

Commit message: fix urdf and fix state representation, action input of GVR (26-D -> 16-D that follows Markovian, flip_vel -> flip_pos)

File: dynamics/resources/gvr_bot/gvrbot_updated.urdf (robot description, URDF)
Before this commit: robot gvrbot_updated, 32 links, 31 joints
Joints:
- removed joint base_to_RF_flipper
- added joint LF_to_RF_flipper: type fixed, parent LF_flipper_main, child RF_flipper_main, origin xyz=0 0.4836 0, axis 0 1 0
- joint base_to_flippers: limit effort=1.0 velocity=1.2 -> (none); origin xyz=0.2605 -0.2418 0.0125 -> xyz=0.2605 -0.2418 0.0125 rpy=0 -3.14 0

Commit message: update GVR model and physics

File: dynamics/resources/gvr_bot/gvrbot_updated.urdf (robot description, URDF)
Before this commit: robot gvrbot_updated, 32 links, 31 joints
Links:
- added link box, mass 0; visual box size=0.1 0.1 0.1
Joints:
- added joint box_link: type fixed, parent base_link, child box, origin xyz=0 0 0.3
