Commit message: add support for customized terrain from LINC

File: dynamics/resources/gvr_bot/test_track/Cliff/cliff.urdf (robot description, URDF)
Before this commit: robot chicane_robot, 2 links, 1 joints
Links:
- removed link chicane
- added link cliff, mass 10.0; collision mesh filename=terrain_cliff.stl scale=1 1 1; visual mesh filename=terrain_cliff.stl scale=1 1 1
Joints:
- joint ramp_to_plane: child chicane -> cliff

File: dynamics/resources/gvr_bot/test_track/Potholes/potholes.urdf (robot description, URDF)
Before this commit: robot chicane_robot, 2 links, 1 joints
Links:
- removed link chicane
- added link potholes, mass 10.0; collision mesh filename=terrain_potholes.stl scale=1 1 1; visual mesh filename=terrain_potholes.stl scale=1 1 1
Joints:
- joint ramp_to_plane: child chicane -> potholes

File: dynamics/resources/gvr_bot/test_track/Stairs/stairs.urdf (robot description, URDF)
Before this commit: robot chicane_robot, 2 links, 1 joints
Links:
- removed link chicane
- added link stairs, mass 10.0; collision mesh filename=terrain_stairs.stl scale=1 1 1; visual mesh filename=terrain_stairs.stl scale=1 1 1
Joints:
- joint ramp_to_plane: child chicane -> stairs
